File: ABBlind.sch (KiCad schematic (older format))
At the start: 16 parts

Commit message: Finished v0.1 schematic
Parts:
- added BRD?: ARDUINO_UNO, symbol ARDUINO_UNO
- added C? (x2): 0.1uF, symbol C
- added C?: C, symbol C
- added C?: 1uF X5R, symbol C
- added C?: 0.1-1uF X5R, symbol C
- added SW? (x2): SW_PUSH, symbol SW_PUSH
- added U?: TLV70033DDCT, symbol REGULATORS_TLV700xx
Connections:
- net labels added: +3.3V, +5V, FOOTSWITCH, ~RESET
- wire segments 49 -> 104
- no-connect marks 7 -> 21
Other:
- note added: "TI recommeds a\n0.1uF bypass cap\nnear supply"
- moved on the sheet: U?A, U?B

Commit message: Add footprint and symbol for LED bicolor
Parts:
- removed D? (x3): Led_x2, symbol Led_x2
- removed R? (x4): R, symbol R
- added D1, D2, D3: LED_BICOLOR, symbol LED_BICOLOR
- added R3, R4, R5, R6: R, Resistors_SMD:R_0805_HandSoldering, symbol R
- C1, C2, C3, C4, C5: renamed from C?; footprint (none) -> Capacitors_SMD:C_0805_HandSoldering
- J1, J2, J3: renamed from J?; footprint (none) -> kicad-library:Conn_Jack_Female_635_THD
- R1, R2: renamed from R?; footprint (none) -> Resistors_SMD:R_0805_HandSoldering
- SW1, SW2: renamed from SW?; footprint (none) -> kicad-library:Switches-Push_switch_THD
- U3: renamed from U?; footprint (none) -> kicad-library:SOT-23-5
- gave numbers to parts that had none: 3
Connections:
- wire segments 104 -> 107
- no-connect marks 21 -> 23
Other:
- moved on the sheet: R2
